File: BSBoard/BSBoard.kicad_sch (KiCad schematic)
At the start: 24 parts, among them J1 Power Switch, J2 Battery, Q1 DMG1012T, U1 CMT-1209-590T, U2 MSP3526

Commit message: Um, yeah, abortive attempt at doing an RP2350 based design. Maybe someday?
Parts:
- removed A1: Adafruit_Feather_Generic, Module:Adafruit_Feather, symbol MCU_Module:Adafruit_Feather_Generic
- added C1, C20, C4: 10uF, Capacitor_SMD:C_0805_2012Metric_Pad1.18x1.45mm_HandSolder, symbol Adafruit Feather RP2350-eagle-import:CAP_CERAMIC0805-NOOUTLINE
- added C10, C11, C15, C17: 1uF, Capacitor_SMD:C_0603_1608Metric_Pad1.08x0.95mm_HandSolder, symbol Adafruit Feather RP2350-eagle-import:CAP_CERAMIC_0402NO
- added C12, C14, C16, C18, C22, C6, C7, C9: 0.1uF, Capacitor_SMD:C_0603_1608Metric_Pad1.08x0.95mm_HandSolder, symbol Adafruit Feather RP2350-eagle-import:CAP_CERAMIC_0402NO
- added C13, C8: 10uF, Capacitor_SMD:C_0805_2012Metric_Pad1.18x1.45mm_HandSolder, symbol Adafruit Feather RP2350-eagle-import:CAP_CERAMIC_0603MP
- added C19, C21: 2.2uF, Adafruit Feather RP2350:_0402NO, symbol Adafruit Feather RP2350-eagle-import:CAP_CERAMIC_0402NO
- added C2, C3: 15pF, Capacitor_SMD:C_0603_1608Metric_Pad1.08x0.95mm_HandSolder, symbol Adafruit Feather RP2350-eagle-import:CAP_CERAMIC_0402NO
- added C5: 10uF, Capacitor_SMD:C_0805_2012Metric_Pad1.18x1.45mm_HandSolder, symbol Adafruit Feather RP2350-eagle-import:CAP_CERAMIC0603_NO
- added CHG1: ORANGE, Adafruit Feather RP2350:CHIPLED_0603_NOOUTLINE, symbol Adafruit Feather RP2350-eagle-import:LED0603_NOOUTLINE
- added D17: PMEG2020AEA, Adafruit Feather RP2350:SOD-323F, symbol Adafruit Feather RP2350-eagle-import:DIODESOD-323F
- added DEBUG1: JST_SH3, Adafruit Feather RP2350:JST_SH3_RA, symbol Adafruit Feather RP2350-eagle-import:CON_JST_SH_3PINVERT
- added L1: DFE252012F-3R3M=P2, Adafruit Feather RP2350:INDUCTOR_1007, symbol Adafruit Feather RP2350-eagle-import:INDUCTOR
- added L2: RED, Adafruit Feather RP2350:CHIPLED_0603_NOOUTLINE, symbol Adafruit Feather RP2350-eagle-import:LED0603_NOOUTLINE
- added Q3: DMG3415UFY, Adafruit Feather RP2350:DFN2015-3, symbol Adafruit Feather RP2350-eagle-import:MOSFET-P_DFN2015
- added R10, R21, R4, R5, R7, R8: 10K, Resistor_SMD:R_0603_1608Metric_Pad0.98x0.95mm_HandSolder, symbol Adafruit Feather RP2350-eagle-import:RESISTOR_0402NO
- added R11, R6: 1K, Resistor_SMD:R_0603_1608Metric_Pad0.98x0.95mm_HandSolder, symbol Adafruit Feather RP2350-eagle-import:RESISTOR_0402NO
- added R12, R13, R9: 5.1K, Resistor_SMD:R_0603_1608Metric_Pad0.98x0.95mm_HandSolder, symbol Adafruit Feather RP2350-eagle-import:RESISTOR_0402NO
- added R14: 10, Resistor_SMD:R_0603_1608Metric_Pad0.98x0.95mm_HandSolder, symbol Adafruit Feather RP2350-eagle-import:RESISTOR_0402NO
- added R16, R17: 27 ohm, Resistor_SMD:R_0603_1608Metric_Pad0.98x0.95mm_HandSolder, symbol Adafruit Feather RP2350-eagle-import:RESISTOR_0402NO
- added R3: 200, Resistor_SMD:R_0603_1608Metric_Pad0.98x0.95mm_HandSolder, symbol Adafruit Feather RP2350-eagle-import:RESISTOR_0402NO
- added SJ1: SOLDERJUMPERCLOSED, Adafruit Feather RP2350:SOLDERJUMPER_CLOSEDWIRE, symbol Adafruit Feather RP2350-eagle-import:SOLDERJUMPERCLOSED
- added SW1, SW2: KMR2, Adafruit Feather RP2350:BTN_RKB2_4.6X2.8, symbol Adafruit Feather RP2350-eagle-import:SWITCH_TACT_SMT_RKB2
- added TP3: TESTPOINTROUND1.5MMNO, Adafruit Feather RP2350:TESTPOINT_ROUND_1.5MM_NO, symbol Adafruit Feather RP2350-eagle-import:TESTPOINTROUND1.5MMNO
- added U$31, U$32: MOUNTINGHOLE2.5, Adafruit Feather RP2350:MOUNTINGHOLE_2.5_PLATED, symbol Adafruit Feather RP2350-eagle-import:MOUNTINGHOLE2.5
- added U$34, U$35: FIDUCIAL_1MM, Adafruit Feather RP2350:FIDUCIAL_1MM, symbol Adafruit Feather RP2350-eagle-import:FIDUCIAL_1MM
- added U3: RT9080-3.3, Adafruit Feather RP2350:SOT23-5, symbol Adafruit Feather RP2350-eagle-import:VREG_SOT23-5
- added U4: MCP73831T-2ACI/OT, Adafruit Feather RP2350:SOT23-5, symbol Adafruit Feather RP2350-eagle-import:MCP73831/2
- added U6: 8MB QSPI, Adafruit Feather RP2350:USON8_4X4, symbol Adafruit Feather RP2350-eagle-import:SPIFLASH_8PIN_4X4
- added X1: JSTPH, Adafruit Feather RP2350:JSTPH2_BATT, symbol Adafruit Feather RP2350-eagle-import:CON_JST_PH_2PIN_MT_BATT
- added X2: DNP, Adafruit Feather RP2350:QFN60_7MM_REDUCEDEPAD, symbol Adafruit Feather RP2350-eagle-import:RP2350_QFN60
- added X6: USB Type C, Adafruit Feather RP2350:USB_C_CUSB31-CFM2AX-01-X, symbol Adafruit Feather RP2350-eagle-import:USB_C
- added Y1: 12MHz/10pF/50ohm, Adafruit Feather RP2350:CRYSTAL_2.5X2, symbol Adafruit Feather RP2350-eagle-import:CRYSTAL2.5X2.0
Connections:
- net GND: now also C1.2, C10.2, C11.2, C12.2, C13.2, C14.2, C15.2, C16.2, C17.2, C18.1, C19.2, C2.1, C20.2, C21.2, C22.2, C3.1, C4.2, C5.2, C6.1, C7.1, C8.2, C9.2, DEBUG1.2, DEBUG1.MT1 (MT), DEBUG1.MT2 (MT), L2.C, R12.1, R13.1, R4.1, R9.2, SW1.B (S), SW1.B' (S1), SW2.B (S), SW2.B' (S1), U3.2 (GND), U4.2 (VSS), U6.4 (VSS), U6.PAD (VSS), X1.1, X1.NC1 (P$1), X1.NC2 (P$1), X2.47 (VREG_PGND), X2.P$1 (GND), X6.A1B12 (GND), X6.B1A12 (GND)
- new net: CHG1.C, R8.1
- new net: SJ1.1, U4.3 (VBAT)
- new net: L2.A, R7.2
- new net: C3.2, R6.1, Y1.1
- new net: R6.2, X2.22 (XOUT)
- new net: R8.2, U4.1 (STAT)
- new net: R9.1, U4.5 (PROG)
- new net: C2.2, X2.21 (XIN), Y1.3 (2)
- new net 1.2V: C18.2, C6.2, C7.2, C8.1, L1.P$1 (1), X2.23 (DVDD), X2.39 (DVDD), X2.50 (VREG_FB), X2.6 (DVDD)
- new net 3.3V: C10.1, C11.1, C12.1, C13.1, C14.1, C15.1, C16.1, C17.1, C22.1, C4.1, C5.1, C9.1, R10.2, R14.1, R21.1, R3.2, U3.5 (OUT), U6.8 (VCC), X2.1 (IOVDD), X2.11 (IOVDD), X2.20 (IOVDD), X2.30 (IOVDD), X2.38 (IOVDD), X2.45 (IOVDD), X2.49 (VREG_VIN), X2.53 (USB_OTP_VDD), X2.54 (QSPI_IOVDD)
- new net A0: X2.40 (GPIO26/AD0)
- new net A1: X2.41 (GPIO27/AD1)
- new net A2: X2.42 (GPIO28/AD2)
- new net A3: X2.43 (GPIO29/AD3)
- new net ADC_AVDD: C19.1, R3.1, X2.44 (ADC_AVDD)
- new net CC1: R13.2, X6.A5 (CC1)
- new net CC2: R12.2, X6.B5 (CC2)
- new net D+: R16.2, X2.52 (USB_D+)
- new net D-: R17.2, X2.51 (USB_D-)
- new net D10: X2.14 (SCK1/CTS1/SDA1/PWM5A/GPIO10)
- new net D11: X2.15 (MOSI1/RTS1/SCL1/PWM5B/GPIO11)
- new net D24: X2.36 (GPIO24/MISO1/TX1/SDA0/PWM4A)
- new net D25: X2.37 (GPIO25/CS1/RX1/SCL0/PWM4B/)
- new net D4: X2.7 (MISO0/TX1/SDA0/PWM2A/GPIO4)
- new net D5: X2.8 (CS0/RX1/SCL0/PWM2B/GPIO5)
- new net D6: X2.9 (SCK0/CTS1/SDA1/PWM3A/GPIO6)
- new net D7: R7.1, X2.10 (MOSI0/RTS1/SCL1/PWM3B/GPIO7)
- new net D9: X2.13 (CS1/RX1/SCL0/PWM4B/GPIO9)
- new net EN: R5.1, U3.3 (EN)
- new net HSTX12: X2.16 (HSTX/MISO1/TX0/SDA0/PWM6A/GPIO12)
- new net HSTX13: X2.17 (HSTX/CS1/RX0/SCL0/PWM6B/GPIO13)
- new net HSTX14: X2.18 (HSTX/SCK1/CTS0/SDA1/PWM7A/GPIO14)
- new net HSTX15: X2.19 (HSTX/MOSI1/RTS0/SCL1/PWM7B/GPIO15)
- new net HSTX16: X2.27 (HSTX/MISO0/TX0/SDA0/PWM0A/GPIO16)
- new net HSTX17: X2.28 (HSTX/CS0/RX0/SCL0/PWM0B/GPIO17)
- new net HSTX18: X2.29 (HSTX/SCK0/CTS0/SDA1/PWM1A/GPIO18)
- new net HSTX19: X2.31 (XPI_CS1/HSTX/MOSI0/RTS0/SCL1/PWM1B/GPIO19)
- new net LX: L1.P$2 (2), X2.48 (VREG_LX)
- new net MISO: X2.32 (MISO0/TX1/SDA0/PWM2A/GPIO20)
- new net MOSI: X2.35 (MOSI0/RTS1/SCL1/PWM3B/GPIO23)
- new net NEOPIX: X2.33 (CS0/RX1/SCL0/PWM2B/GPIO21)
- new net PSRAM_CS: X2.12 (XIP_CS1/MISO1/TX1/SDA0/PWM4A/GPIO8)
- new net QSPI_CS: R10.1, R11.1, U6.1 (SSEL), X2.60 (~{QSPI_CS})
- new net QSPI_DATA[0]: U6.5 (MOSI), X2.57 (QSPI_SD0)
- new net QSPI_DATA[1]: U6.2 (MISO), X2.59 (QSPI_SD1)
- new net QSPI_DATA[2]: U6.3 (WP#/IO2), X2.58 (QSPI_SD2)
- new net QSPI_DATA[3]: U6.7 (HOLD#/IO3), X2.55 (QSPI_SD3)
- new net QSPI_SCK: U6.6 (SCK), X2.56 (QSPI_SCLK)
- new net RX: X2.3 (CS0/RX0/SCL0/PWM0B/GPIO1)
- new net SCK: X2.34 (SCK0/CTS1/SDA1/PWM3A/GPIO22)
- new net SCL: X2.5 (MOSI0/RTS0/SCL1/PWM1B/GPIO3)
- new net SDA: X2.4 (SCK0/CTS0/SDA1/PWM1A/GPIO2)
- new net SWCLK: DEBUG1.1, X2.24 (SWCLK)
- new net SWDIO: DEBUG1.3, X2.25 (SWDIO)
- new net TX: X2.2 (XPI_CS1/MISO0/TX0/SDA0/PWM0A/GPIO0)
- new net USBBOOT: R11.2, SW2.A (P), SW2.A' (P1), TP3.P$1
- new net USB_D+: R16.1, X6.A6 (D+), X6.B6 (D+)
- new net USB_D-: R17.1, X6.A7 (D-), X6.B7 (D-)
- new net VBAT: C20.1, Q3.3 (D), SJ1.2, X1.2
- new net VBUS: CHG1.A, D17.A, Q3.1 (G), R4.2, U4.4 (VDD), X6.A4B9 (VBUS), X6.B4A9 (VBUS)
- new net VHI: C1.1, D17.C, Q3.2 (S), R5.2, U3.1 (IN)
- new net VREG_AVDD: C21.1, R14.2, X2.46 (VREG_AVDD)
- new net ~{RESET}: R21.2, SW1.A (P), SW1.A' (P1), X2.26 (/RUN)
Other:
- note added: "1.0K = 1000mA"
- note added: "10K = 100mA"
- note added: "2.0K = 500mA"
- note added: "5.0K = 200mA"
- note added: "POWER AND FILTERING"
- note added: "RED LED"
- note added: "RESET"
- note added: "USB AND BATTERY CHARGING"
- moved on the sheet: D1, D10, D11, D12, D13, D14, D15, D2, D3, D4, D5, D6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
